File: pcb files/signal detector.kicad_pcb (KiCad board)
At the start: 2 copper layers, 67 x 150.5 mm, 57 parts, among them J1 USB_C_Receptacle_USB2.0_16P, J2 Conn_01x05_Pin, J3 Conn_Coaxial, M1 Motor_DC, Q1 2N7002, Q2 2N7002, Q3 2N7002, SW1 SW_Push, SW2 SW_SPST, SW3 SW_Push, SW5 RotaryEncoder_Switch, U1 MCP73831-2-MC, U2 AP2112K-3.3, U3 CR2013-MI2120, U4 ESP32-C3-WROOM-02, U5 AD8318ACPZ-REEL7, U6 PCA9536D

Commit message: Add files via upload
Parts:
- R18: footprint Resistor_SMD:R_2512_6332Metric -> Resistor_SMD:R_0805_2012Metric
- moved R4 7.50 mm to (153.0, 173.0)
- moved SW5 4.79 mm to (91.5, 165.0)
- moved SW1 3.00 mm to (152.0, 165.9), turned to -90 degrees
Connections:
- J1 pad A6: unconnected-(J1-D+-PadA6) -> /USB_P
- J1 pad A7: unconnected-(J1-D--PadA7) -> /USB_N
- J1 pad B6: /USB D+ -> /USB_P
- J1 pad B7: /USB D− -> /USB_N
- U4 pad 13: /USB D− -> /USB_N
- U4 pad 14: /USB D+ -> /USB_P
Routing:
- net Net-(U4-EN): track 130.9 -> 105.2 mm, vias 2 -> 4
- net /GPIO_10: track 79.9 -> 97.8 mm, vias 5 -> 3
- net /USB_P: track 0.00 -> 17.6 mm
- net /USB_N: track 0.00 -> 17.0 mm
- net /USB D+: track 15.6 -> 0.00 mm
- net Net-(U3-D/~{C}): track 85.5 -> 71.7 mm
- net /USB D−: track 13.5 -> 0.00 mm
- net Net-(U1-PROG): track 24.4 -> 13.0 mm, vias 0 -> 2
- net Net-(U3-SCK): track 76.6 -> 66.7 mm, vias 0 -> 1
- net GND: track 378.0 -> 369.5 mm, vias 34 -> 30
- net /VBAT_SYS: track 74.1 -> 81.6 mm, vias 5 -> 3
- net +5V: track 78.8 -> 71.9 mm, vias 10 -> 4
- net /IO0: track 13.4 -> 17.9 mm, vias 2 -> 1
- net /IO1: track 57.1 -> 60.0 mm, vias 2 -> 1
- net Net-(BZ1--): track 21.6 -> 19.2 mm, vias 0 -> 1
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- added copper zone on B.Cu, net GND
- added copper zone on F.Cu, net GND
Other:
- board size 67 x 150.5 mm -> 71 x 150.5 mm
